File: original/schaltung/pc880.kicad_sch (KiCad schematic)
At the start: 0 parts

Commit message: Schaltplantitel
Other:
- title: (none) -> Polycomputer 880
Changed lines of the file:
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@@
 (kicad_sch (version 20230121) (generator eeschema)
   (paper "A4")
+  (title_block
+    (title "Polycomputer 880")
+  )
   (junction (at 54.61 162.56) (diameter 0) (color 0 0 0 0)
   )
