File: original/schaltung/clock.kicad_sch (KiCad schematic)
At the start: 41 parts, among them K1 RESET, K2 MON, K3 MCYCL, K4 CYCL, Q1 7.3728M, T1 SS216

Commit message: Schönheitskorrekturen Schaltplan
Parts:
- renumbered C25 to C27, C25 to C7, C25 to C8
