File: original/schaltung/cpu.kicad_sch (KiCad schematic)
At the start: 36 parts, among them U1 U880D

Commit message: Schönheitskorrekturen Schaltplan
Parts:
- renumbered U1 to I1
Connections:
- net +5V: now also I1.11 (Vcc)
- net GND: now also I1.29 (GND)
