File: original/schaltung/disp.kicad_sch (KiCad schematic)
At the start: 71 parts, among them T17 SS216, T18 SS216, T19 KFY18, T20 KFY18, T21 KFY18, T22 KFY18, T23 KFY18, T24 KFY18, T25 KFY18, T26 KFY18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

Commit message: Schönheitskorrekturen Schaltplan
Parts:
- renumbered C25 to C36, C25 to C37
